File: tinyG2Hat.brd (EAGLE design)
At the start: 102.6 x 69.1 mm, 31 parts

Commit message: Début de la sérigraphie
Parts:
- SPINDLE_OUTPUTS: device con-lstb:MA05-2 -> pinhead:2X05
- SV1: device con-lstb:MA04-2 -> pinhead:2X04
- moved S2 1.27 mm to (75.4, 59.7)
Routing:
- net Z_MIN: track 6.12 -> 4.85 mm
- net Z_MAX: track 6.12 -> 4.85 mm
- net Y_MIN: track 6.12 -> 4.85 mm
- net Y_MAX: track 6.12 -> 4.85 mm
- net X_MIN: track 6.12 -> 4.85 mm
- net X_MAX: track 6.12 -> 4.85 mm
- net N$53: track 25.1 -> 24.6 mm
- net N$55: track 29.5 -> 29.0 mm
- net N$51: track 20.6 -> 20.1 mm
- net H_INTERLCK: track 97.6 -> 97.1 mm
- net N$49: track 15.2 -> 14.7 mm
- net E_STOP: track 173.8 -> 173.3 mm
Other:
- board text added: "CTRL"
- board text added: "LCK"
- board text added: "STOP"
- board text added: "X"
- board text added: "Xmax"
- board text added: "Xmin"
- board text added: "Y"
- board text added: "Ymax"
- board text added: "Ymin"
- board text added: "Z"
- board text added: "Zmax"
- board text added: "Zmin"

Commit message: Sérigraphie finie
Parts:
- added U$7: (no value), Aliom:OPEN_HARDWARE_5MM
- added U$8: (no value), Aliom:LABSUD_15MM
- S2: device switch-dil:DP-08 -> switch-dil:DIP08YL
- moved CONTROL_SWITCHES_INPUTS 0.36 mm to (6.86, 28.4)
Routing:
- net N$50: track 27.1 -> 27.6 mm
Other:
- board size 102.6 x 69.1 mm -> 102.6 x 68.8 mm
- board text added: "+24V"
- board text added: "Coolant"
- board text added: "Dir"
- board text added: "Emergency Stop"
- board text added: "Enable"
- board text added: "Feed-Hold"
- board text added: "Lucas MOLIA & Renaud ADNET"
- board text added: "Mot 1"
- board text added: "Mot 2"
- board text added: "Mot 3"
- board text added: "Mot 4"
- board text added: "Mot 5"
- board text added: "Mot 6"
- board text added: "PWM"
- board text added: "PWM 2"
- board text added: "Reset"
- board text added: "Soft-Reset"
- board text added: "Spindle"
- board text added: "Step config"
- board text added: "Y-start"
- board text added: "____________"
- board text added: "____________ |Full | 0 | 0 | 0 | |1/2 | 1 | 0 | 0 | |1/4 | 0 | 1 | 0 | |1/8 | 1 | 1 | 0 | |1/16 | 0 | 0 | 1 | |1/32 | 1 | 1 | 1 |"
