File: tinyG2Hat.brd (EAGLE design)
At the start: 102.6 x 68.8 mm, 33 parts

Commit message: Finalisation
Other:
- board size 102.6 x 68.8 mm -> 101.9 x 68.8 mm
Changed lines of the file:
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@@
 <wire x1="-0.254" y1="56.134" x2="-0.254" y2="1.778" width="0" layer="20"/>
 <wire x1="1.524" y1="0.254" x2="98.806" y2="0.254" width="0" layer="20"/>
-<wire x1="99.822" y1="1.27" x2="99.822" y2="3.556" width="0" layer="20"/>
-<wire x1="99.822" y1="3.556" x2="102.362" y2="6.096" width="0" layer="20"/>
-<wire x1="102.362" y1="6.096" x2="102.362" y2="38.862" width="0" layer="20"/>
-<wire x1="102.362" y1="38.862" x2="99.822" y2="41.402" width="0" layer="20"/>
-<wire x1="99.822" y1="41.402" x2="99.822" y2="52.832" width="0" layer="20"/>
+<wire x1="99.822" y1="1.27" x2="99.822" y2="4.064" width="0" layer="20"/>
+<wire x1="99.822" y1="4.064" x2="101.6" y2="5.842" width="0" layer="20"/>
+<wire x1="101.6" y1="5.842" x2="101.6" y2="38.862" width="0" layer="20"/>
+<wire x1="101.6" y1="38.862" x2="99.822" y2="40.64" width="0" layer="20"/>
 <wire x1="62.23" y1="56.896" x2="0.762" y2="56.896" width="0" layer="20"/>
 <wire x1="0.762" y1="56.896" x2="-0.254" y2="56.134" width="0" layer="20" curve="90"/>
 <wire x1="-0.254" y1="1.778" x2="1.524" y2="0.254" width="0" layer="20" curve="90"/>
 <wire x1="98.806" y1="0.254" x2="99.822" y2="1.27" width="0" layer="20" curve="90"/>
-<wire x1="99.822" y1="52.832" x2="99.822" y2="67.818" width="0" layer="20"/>
+<wire x1="99.822" y1="40.64" x2="99.822" y2="67.818" width="0" layer="20"/>
 <wire x1="99.822" y1="67.818" x2="98.552" y2="69.088" width="0" layer="20"/>
 <wire x1="98.552" y1="69.088" x2="64.262" y2="69.088" width="0" layer="20"/>
@@
 <text x="60.706" y="20.32" size="0.6096" layer="21" rot="R90" align="center">100µF</text>
 <text x="35.306" y="20.066" size="0.6096" layer="21" rot="R90" align="center">100µF</text>
+<dimension x1="103.632" y1="0.254" x2="103.632" y2="68.834" x3="105.664" y3="34.544" textsize="1.778" layer="20"/>
+<dimension x1="-0.254" y1="-2.54" x2="101.6" y2="-2.54" x3="50.673" y3="-3.302" textsize="1.778" layer="20"/>
 </plain>
 <attributes>

Commit message: Finalisation
Other:
- board size 101.9 x 68.8 mm -> 100.1 x 68.8 mm
Changed lines of the file:
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@@
 <wire x1="-0.254" y1="56.134" x2="-0.254" y2="1.778" width="0" layer="20"/>
 <wire x1="1.524" y1="0.254" x2="98.806" y2="0.254" width="0" layer="20"/>
-<wire x1="99.822" y1="1.27" x2="99.822" y2="4.064" width="0" layer="20"/>
-<wire x1="99.822" y1="4.064" x2="101.6" y2="5.842" width="0" layer="20"/>
-<wire x1="101.6" y1="5.842" x2="101.6" y2="38.862" width="0" layer="20"/>
-<wire x1="101.6" y1="38.862" x2="99.822" y2="40.64" width="0" layer="20"/>
 <wire x1="62.23" y1="56.896" x2="0.762" y2="56.896" width="0" layer="20"/>
 <wire x1="0.762" y1="56.896" x2="-0.254" y2="56.134" width="0" layer="20" curve="90"/>
 <wire x1="-0.254" y1="1.778" x2="1.524" y2="0.254" width="0" layer="20" curve="90"/>
 <wire x1="98.806" y1="0.254" x2="99.822" y2="1.27" width="0" layer="20" curve="90"/>
-<wire x1="99.822" y1="40.64" x2="99.822" y2="67.818" width="0" layer="20"/>
 <wire x1="99.822" y1="67.818" x2="98.552" y2="69.088" width="0" layer="20"/>
 <wire x1="98.552" y1="69.088" x2="64.262" y2="69.088" width="0" layer="20"/>
@@
 <text x="35.306" y="20.066" size="0.6096" layer="21" rot="R90" align="center">100µF</text>
 <dimension x1="103.632" y1="0.254" x2="103.632" y2="68.834" x3="105.664" y3="34.544" textsize="1.778" layer="20"/>
-<dimension x1="-0.254" y1="-2.54" x2="101.6" y2="-2.54" x3="50.673" y3="-3.302" textsize="1.778" layer="20"/>
+<wire x1="99.822" y1="1.27" x2="99.822" y2="67.818" width="0" layer="20"/>
+<dimension x1="-0.254" y1="-4.064" x2="99.822003125" y2="-4.064" x3="49.784" y3="-4.064" textsize="1.778" layer="20" dtype="radius"/>
 </plain>
 <attributes>
